File: hardware/StepStick-Protector_v11.brd (EAGLE design)
At the start: 15.2 x 20.3 mm, 15 parts, among them IC1 STEPSTICK-TP, J1 JUMPER2-0603-NC, X1 PASSER, X2 PASSER

Commit message: updated schematics and layout files
Parts:
- D1+, D1-, D2+, D2-, D3+, D3-, D4+, D4-: value (none) -> S310FA; device we-rcl:SMA_DO214AC -> we-rcl:SOD123
- moved D4- 0.89 mm to (4.13, 6.92), turned to 180 degrees
- moved C1 0.57 mm to (5.17, 2.34)
Routing:
- net GND: track 2.73 -> 0.00 mm
- net M1B: track 11.4 -> 13.1 mm
- net VM: track 28.1 -> 26.7 mm
