File: hardware/SilentStepStick-TMC5160_v14.brd (EAGLE design)
At the start: 15.2 x 20.3 mm, 40 parts, among them IC1 TMC5160-WA, IC2 FDMC8030, IC3 FDMC8030, IC4 FDMC8030, IC5 FDMC8030, P1 MA08-1, P2 MA08-1, P3 MA02-1, X1 PASSER-04, X2 PASSER-04, X3 PASSER-04, X4 PASSER-04

Commit message: updated schematics
Connections:
- net N$11 renamed SD_MODE
- net N$3 renamed 12VOUT
- net N$41 renamed DCEN
- net N$44 renamed SPI_MODE
Changed lines of the file:
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@@
 <wire x1="6.9416" y1="5.0227" x2="6.7" y2="5.1143" width="0.2" layer="1"/>
 </signal>
-<signal name="N$3">
+<signal name="12VOUT">
 <contactref element="IC1" pad="4"/>
 <contactref element="C3" pad="2"/>
@@
 <wire x1="4.87" y1="5.952975" x2="4.87" y2="6.235" width="0.1524" layer="1"/>
 </signal>
-<signal name="N$41">
+<signal name="DCEN">
 <contactref element="IC1" pad="23"/>
 <contactref element="DCEN" pad="2"/>
@@
 <wire x1="2.5092" y1="13.95" x2="1.27" y2="13.95" width="0.2" layer="4"/>
 </signal>
-<signal name="N$11">
+<signal name="SD_MODE">
 <contactref element="IC1" pad="21"/>
 <contactref element="SD_MODE" pad="2"/>
@@
 <wire x1="2.2582" y1="4.1973" x2="2.7305" y2="3.725" width="0.1524" layer="1"/>
 </signal>
-<signal name="N$44">
+<signal name="SPI_MODE">
 <contactref element="IC1" pad="22"/>
 <wire x1="3.655" y1="8.45" x2="3.695" y2="8.41" width="0.2" layer="1"/>
