File: hardware/SilentStepStick-TMC5160_v14.sch (EAGLE design)
At the start: 40 parts, among them IC1 TMC5160-WA, IC2 FDMC8030, IC3 FDMC8030, IC4 FDMC8030, IC5 FDMC8030, P1 MA08-1, P2 MA08-1, P3 MA02-1, X1 PASSER-04, X2 PASSER-04, X3 PASSER-04, X4 PASSER-04

Commit message: updated schematics
Connections:
- net N$11 renamed SD_MODE
- net N$3 renamed 12VOUT
- net N$41 renamed DCEN
- net N$44 renamed SPI_MODE
Changed lines of the file:
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@@
 <setting verticaltext="up"/>
 </settings>
-<grid distance="0.05" unitdist="inch" unit="inch" style="lines" multiple="1" display="yes" altdistance="0.01" altunitdist="inch" altunit="inch"/>
+<grid distance="0.1" unitdist="inch" unit="inch" style="lines" multiple="1" display="no" altdistance="0.01" altunitdist="inch" altunit="inch"/>
 <layers>
 <layer number="1" name="Top" color="4" fill="1" visible="no" active="no"/>
@@
 </segment>
 </net>
-<net name="N$3" class="0">
+<net name="12VOUT" class="0">
 <segment>
 <pinref part="IC1" gate="G$1" pin="12VOUT"/>
@@
 </segment>
 </net>
-<net name="N$41" class="0">
+<net name="DCEN" class="0">
 <segment>
 <pinref part="IC1" gate="G$1" pin="ENCB_DCEN_CFG4"/>
@@
 </segment>
 </net>
-<net name="N$11" class="0">
+<net name="SD_MODE" class="0">
 <segment>
 <pinref part="IC1" gate="G$1" pin="SD_MODE"/>
@@
 </segment>
 </net>
-<net name="N$44" class="0">
+<net name="SPI_MODE" class="0">
 <segment>
 <pinref part="IC1" gate="G$1" pin="SPI_MODE"/>
